File: MPCNC Nano Estlcam Shield.sch (KiCad schematic (older format))
At the start: 81 parts, among them J1 Screw_Terminal_01x02, J10 Conn_01x04_Male, J11 Conn_01x04_Male, J12 Screw_Terminal_01x03, J13 Screw_Terminal_01x03, J14 Screw_Terminal_01x03, J15 Conn_02x03_Odd_Even, J16 Screw_Terminal_01x02, J17 Screw_Terminal_01x02, J18 Screw_Terminal_01x03, J19 Screw_Terminal_01x03, J2 Conn_01x03_Male, J20 Screw_Terminal_01x03, J21 Screw_Terminal_01x03, J22 Screw_Terminal_01x03, J23 Screw_Terminal_01x03, J24 Screw_Terminal_01x03, J25 Screw_Terminal_01x03, J26 Screw_Terminal_01x03, J27 Screw_Terminal_01x03, J28 Conn_01x03_Female, J3 Conn_01x06_Male, J4 Screw_Terminal_01x03, J5 Screw_Terminal_01x03, J6 Screw_Terminal_01x03, J7 Conn_01x04_Male, J8 Conn_01x04_Male, J9 Conn_01x04_Male, U1 LM358, U2 LTV-847, U3 LTV-847, U4 LTV-847, U5 ULN2003, U6 L7805, U7 ATtiny45-20PU

Commit message: V1.2
- Version 1.2 of MPCNC Nano Estlcam Shield
   PCB schematic changes:
    + Power LEDs (5mm LED) added(5V and VMot[formerly VDD])
    + 3,3V connector added
    + Output Enabled LEDs added (3 x 3mm LED + 1k resistor for OUT1,2,3), Pulls down ouput signal on startup
    # Replaced powerflag "VDD" with "VMot" (new custom symbol)
    + Added net names for Microstepping jumper
    # Signal "Analog_0_5V" now connected to "LM358 +"-Pin net (after instead of before LP-filter)
    # Replaced servo connector symbol (Conn_01x03_Female to Conn_01x03_Male)
    # Mirrored Microstepping and FLT jumper (Pin 1:5V, Pin 2:Signal)
    # Changed net names ("Ex"-> "INx", "Ax" -> "OUTx")
   PCB layout changes:
    # Silk screen text input/output description corrected ("Feedrate" and "E5")
    # Changed silk screen text language to English ("Ex"-> "INx", "Ax" -> "OUTx")
    # Moved traces and parts for schematic changes and increased margin
    # Added silk screen text for some parts (Arduino Nano, LM2596 step down module, Driver modules, Microstepping Jumper, Fan, 0-10V Adjustment Poti and LEDs)
    # Revised LM2596 module footprint
    # Replaced RV1 Trimmer/Potentiometer Footprint (Potentiometer_Bourns_3296Y_Vertical -> Potentiometer_Bourns_3296W_Vertical). Footprint (2 Pads) of Potentiometer_Bourns_3296Y_Vertical is still on PCB. -> It is possible to mount either potentiometer.
    # Changed TerminalBlocks footprint and pin pitch (5.08mm -> 5.00mm)
   Library changes:
    + Added power flag "VMot"
    # Renamed "DCDC_LM2596_Step_Down_Module" to "LM2596_Step_Down_Module"
    + Added modified footprints from KiCAD standard library for some components (Arduino Nano, Terminal blocks, Pololu driver breakout board, Bourns 3296W potentiomter, Heatsink for L7805) (added 3D models to footprint. However, 3D models are not published in repository for licensing reasons)
Parts:
- added D1: LED GREEN, LED_THT:LED_D5.0mm, symbol Device:LED
- added D4: LED RED, LED_THT:LED_D5.0mm, symbol Device:LED
- added D5, D6, D7: LED RED, LED_THT:LED_D3.0mm, symbol Device:LED
- added J29: Conn_01x02_Male, Connector_PinHeader_2.54mm:PinHeader_1x02_P2.54mm_Vertical, symbol Connector:Conn_01x02_Male
- added R14: 220, Resistor_THT:R_Axial_DIN0207_L6.3mm_D2.5mm_P7.62mm_Horizontal, symbol Device:R_Small
- added R15: 1.8k, Resistor_THT:R_Axial_DIN0207_L6.3mm_D2.5mm_P7.62mm_Horizontal, symbol Device:R_Small
- added R16, R17, R18: 1k, Resistor_THT:R_Axial_DIN0207_L6.3mm_D2.5mm_P7.62mm_Horizontal, symbol Device:R_Small
- A1: footprint Module:Arduino_Nano -> MPCNC_Shield_Footprints:Arduino_Nano
- A2, A3, A4: footprint Module:Pololu_Breakout-16_15.2x20.3mm -> MPCNC_Shield_Footprints:Pololu_Breakout-16_15.2x20.3mm
- A5: footprint MPCNC_Shield_Footprints:LM2596_Step_Down_Module-4_21.2x40.3mm -> MPCNC_Shield_Footprints:LM2596_Step_Down_Module-21.3x43.6mm
- C6: value 0.1µF -> 1µF
- HS1: footprint Power_Module:Heatsink_China_TO220_(22x)15x10mm_1xDrill1.5mm -> MPCNC_Shield_Footprints:Heatsink_China_TO220_(22x)15x10mm_1xDrill1.5mm
- J1, J16, J17: footprint TerminalBlock_Phoenix:TerminalBlock_Phoenix_MKDS-1,5-2-5.08_1x02_P5.08mm_Horizontal -> MPCNC_Shield_Footprints:TerminalBlock_RND_205-00012_1x02_P5.00mm_Horizontal
- J12, J13, J14, J18, J19, J20, J21, J22, J23, J24, J25, J4, J5, J6: footprint TerminalBlock_Phoenix:TerminalBlock_Phoenix_MKDS-1,5-3-5.08_1x03_P5.08mm_Horizontal -> MPCNC_Shield_Footprints:TerminalBlock_RND_205-00013_1x03_P5.00mm_Horizontal
- J26: footprint TerminalBlock_Phoenix:TerminalBlock_Phoenix_MKDS-1,5-3-5.08_1x03_P5.08mm_Horizontal -> MPCNC_Shield_Footprints:TerminalBlock_RND_205-00013_1x03_P5.00mm_Horizontal; Funktion Feedrate -> Feedrate Adjust
- J27: footprint TerminalBlock_Phoenix:TerminalBlock_Phoenix_MKDS-1,5-3-5.08_1x03_P5.08mm_Horizontal -> MPCNC_Shield_Footprints:TerminalBlock_RND_205-00013_1x03_P5.00mm_Horizontal; Funktion Rot. Speed -> Rot. Speed Adjust
- J28: value Conn_01x03_Female -> Conn_01x03_Male; symbol Connector:Conn_01x03_Female -> Connector:Conn_01x03_Male
- JP13, JP14: value Jumper_NC_Dual -> Jumper_3_Open; symbol Device:Jumper_NC_Dual -> Jumper:Jumper_3_Open
- RV1: footprint Potentiometer_THT:Potentiometer_Bourns_3296Y_Vertical -> MPCNC_Shield_Footprints:Potentiometer_Bourns_3296W_Vertical
- renumbered D1 to D2, D2 to D3
Connections:
- net +5V: now also JP1.1, JP10.1, JP11.1, JP12.1, JP2.1, JP3.1, JP4.1, JP5.1, JP6.1, JP7.1, JP8.1, JP9.1, D1.2 (A); no longer JP1.2, JP10.2, JP11.2, JP12.2, JP2.2, JP3.2, JP4.2, JP5.2, JP6.2, JP7.2, JP8.2, JP9.2
- net A1(D3): now also R16.1
- net A2(D2): now also R17.1
- net A3(D4): now also R18.2
- net FLT_X: now also JP4.2; no longer JP4.1
- net FLT_Y: now also JP8.2; no longer JP8.1
- net FLT_Z: now also JP12.2; no longer JP12.1
- net GND: now also D5.1 (K), D6.1 (K), D7.1 (K), J29.2 (Pin_2), R14.1, R15.2
- net +3V3: now reaches A1.17 (3V3)
- net +3V3: now also J29.1 (Pin_1)
- net M0X: now reaches A2.10 (M0)
- net M0X: now also JP1.2; no longer JP1.1
- net M1X: now reaches A2.11 (M1)
- net M1X: now also JP2.2; no longer JP2.1
- net M2X: now reaches A2.12 (M2)
- net M2X: now also JP3.2; no longer JP3.1
- net SPINDEL_ON_OFF_R_LED: now reaches R4.2, U4.2
- net Spindle_Speed_Analog_0-5V: now reaches C1.1, JP17.2, R1.2, U1.5 (+)
- net Spindle_Speed_Analog_0-5V: now also U7.3 (XTAL2/PB4)
- net C1_to_JP16: now reaches C1.2, JP16.1
- net RV1_R2: now reaches R2.2, RV1.3
- net R3_RV1: now reaches R3.1, RV1.1
- net M0Y: now reaches A3.10 (M0)
- net M0Y: now also JP5.2; no longer JP5.1
- net M1Y: now reaches A3.11 (M1)
- net M1Y: now also JP6.2; no longer JP6.1
- net M2Y: now reaches A3.12 (M2)
- net M2Y: now also JP7.2; no longer JP7.1
- net M0Z: now reaches A4.10 (M0)
- net M0Z: now also JP9.2; no longer JP9.1
- net M1Z: now reaches A4.11 (M1)
- net M1Z: now also JP10.2; no longer JP10.1
- net M2Z: now reaches A4.12 (M2)
- net M2Z: now also JP11.2; no longer JP11.1
- net +VDC renamed VDC
- net A1 renamed OUT1
- net A2 renamed OUT2
- net A3 renamed OUT3
- net Analog_0-5V|PWM renamed Spindle_PWM(D5)
- net Spindle_PWM(D5): no longer U7.3 (XTAL2/PB4)
- net E1 renamed IN1
- net E1_R_LED renamed IN1_R_LED
- net E2 renamed IN2
- net E2_R_LED renamed IN2_R_LED
- net E3 renamed IN3
- net E3_R_LED renamed IN3_R_LED
- net E4 renamed IN4
- net E4_R_LED renamed IN4_R_LED
- net E5 renamed IN5
- net E5_R_LED renamed IN5_R_LED
- net E6 renamed IN6
- net E6_R_LED renamed IN6_R_LED
- net E7 renamed IN7
- net E7_R_LED renamed IN7_R_LED
- net E8 renamed IN8
- net E8_R_LED renamed IN8_R_LED
- net VDD renamed VMot
- net VMot: now also D4.2 (A)
- new net D1_R_LED: D1.1 (K), R14.2
- new net D4_R_LED: D4.1 (K), R15.1
- new net D5_R_LED: D5.2 (A), R16.2
- new net D6_R_LED: D6.2 (A), R17.2
- new net D7_R_LED: D7.2 (A), R18.1
- no-connect marks 15 -> 13
Other:
- note added: "Variable Frequency Drive 0-10V Speed Control(VI/ACM Input)\nFrequenzumrichter 0-10V Drehzahleinstellung (VI/ACM Eingang)\n\n"
- note removed: "Variable Frequency Drive 0-10V Speed Adjust (VI/ACM Input)\nFrequenzumrichter 0-10V Drehzahleinstellung (VI/ACM Eingang)\n\n"
- moved on the sheet: A1, A2, A3, A4, A5, C1, C2, C3, C4, C5, C6, C7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

Commit message: Revert "V1.2"
This reverts commit 25746ea092c74b1b8c6b498096b07c9fdffcdb93.
Parts:
- removed D1: LED GREEN, LED_THT:LED_D5.0mm, symbol Device:LED
- removed D4: LED RED, LED_THT:LED_D5.0mm, symbol Device:LED
- removed D5, D6, D7: LED RED, LED_THT:LED_D3.0mm, symbol Device:LED
- removed J29: Conn_01x02_Male, Connector_PinHeader_2.54mm:PinHeader_1x02_P2.54mm_Vertical, symbol Connector:Conn_01x02_Male
- removed R14: 220, Resistor_THT:R_Axial_DIN0207_L6.3mm_D2.5mm_P7.62mm_Horizontal, symbol Device:R_Small
- removed R15: 1.8k, Resistor_THT:R_Axial_DIN0207_L6.3mm_D2.5mm_P7.62mm_Horizontal, symbol Device:R_Small
- removed R16, R17, R18: 1k, Resistor_THT:R_Axial_DIN0207_L6.3mm_D2.5mm_P7.62mm_Horizontal, symbol Device:R_Small
- A1: footprint MPCNC_Shield_Footprints:Arduino_Nano -> Module:Arduino_Nano
- A2, A3, A4: footprint MPCNC_Shield_Footprints:Pololu_Breakout-16_15.2x20.3mm -> Module:Pololu_Breakout-16_15.2x20.3mm
- A5: footprint MPCNC_Shield_Footprints:LM2596_Step_Down_Module-21.3x43.6mm -> MPCNC_Shield_Footprints:LM2596_Step_Down_Module-4_21.2x40.3mm
- C6: value 1µF -> 0.1µF
- HS1: footprint MPCNC_Shield_Footprints:Heatsink_China_TO220_(22x)15x10mm_1xDrill1.5mm -> Power_Module:Heatsink_China_TO220_(22x)15x10mm_1xDrill1.5mm
- J1, J16, J17: footprint MPCNC_Shield_Footprints:TerminalBlock_RND_205-00012_1x02_P5.00mm_Horizontal -> TerminalBlock_Phoenix:TerminalBlock_Phoenix_MKDS-1,5-2-5.08_1x02_P5.08mm_Horizontal
- J12, J13, J14, J18, J19, J20, J21, J22, J23, J24, J25, J4, J5, J6: footprint MPCNC_Shield_Footprints:TerminalBlock_RND_205-00013_1x03_P5.00mm_Horizontal -> TerminalBlock_Phoenix:TerminalBlock_Phoenix_MKDS-1,5-3-5.08_1x03_P5.08mm_Horizontal
- J26: footprint MPCNC_Shield_Footprints:TerminalBlock_RND_205-00013_1x03_P5.00mm_Horizontal -> TerminalBlock_Phoenix:TerminalBlock_Phoenix_MKDS-1,5-3-5.08_1x03_P5.08mm_Horizontal; Funktion Feedrate Adjust -> Feedrate
- J27: footprint MPCNC_Shield_Footprints:TerminalBlock_RND_205-00013_1x03_P5.00mm_Horizontal -> TerminalBlock_Phoenix:TerminalBlock_Phoenix_MKDS-1,5-3-5.08_1x03_P5.08mm_Horizontal; Funktion Rot. Speed Adjust -> Rot. Speed
- J28: value Conn_01x03_Male -> Conn_01x03_Female; symbol Connector:Conn_01x03_Male -> Connector:Conn_01x03_Female
- JP13, JP14: value Jumper_3_Open -> Jumper_NC_Dual; symbol Jumper:Jumper_3_Open -> Device:Jumper_NC_Dual
- RV1: footprint MPCNC_Shield_Footprints:Potentiometer_Bourns_3296W_Vertical -> Potentiometer_THT:Potentiometer_Bourns_3296Y_Vertical
- renumbered D2 to D1, D3 to D2
Connections:
- net +5V: now also JP1.2, JP10.2, JP11.2, JP12.2, JP2.2, JP3.2, JP4.2, JP5.2, JP6.2, JP7.2, JP8.2, JP9.2; no longer JP1.1, JP10.1, JP11.1, JP12.1, JP2.1, JP3.1, JP4.1, JP5.1, JP6.1, JP7.1, JP8.1, JP9.1
- net FLT_X: now also JP4.1; no longer JP4.2
- net FLT_Y: now also JP8.1; no longer JP8.2
- net FLT_Z: now also JP12.1; no longer JP12.2
- net +3V3: no longer names the net of A1.17 (3V3)
- net C1_to_JP16: no longer names the net of C1.2, JP16.1
- net IN1 renamed E1
- net IN1_R_LED renamed E1_R_LED
- net IN2 renamed E2
- net IN2_R_LED renamed E2_R_LED
- net IN3 renamed E3
- net IN3_R_LED renamed E3_R_LED
- net IN4 renamed E4
- net IN4_R_LED renamed E4_R_LED
- net IN5 renamed E5
- net IN5_R_LED renamed E5_R_LED
- net IN6 renamed E6
- net IN6_R_LED renamed E6_R_LED
- net IN7 renamed E7
- net IN7_R_LED renamed E7_R_LED
- net IN8 renamed E8
- net IN8_R_LED renamed E8_R_LED
- net M0X: no longer names the net of A2.10 (M0)
- net M0X: now also JP1.1; no longer JP1.2
- net M0Y: no longer names the net of A3.10 (M0)
- net M0Y: now also JP5.1; no longer JP5.2
- net M0Z: no longer names the net of A4.10 (M0)
- net M0Z: now also JP9.1; no longer JP9.2
- net M1X: no longer names the net of A2.11 (M1)
- net M1X: now also JP2.1; no longer JP2.2
- net M1Y: no longer names the net of A3.11 (M1)
- net M1Y: now also JP6.1; no longer JP6.2
- net M1Z: no longer names the net of A4.11 (M1)
- net M1Z: now also JP10.1; no longer JP10.2
- net M2X: no longer names the net of A2.12 (M2)
- net M2X: now also JP3.1; no longer JP3.2
- net M2Y: no longer names the net of A3.12 (M2)
- net M2Y: now also JP7.1; no longer JP7.2
- net M2Z: no longer names the net of A4.12 (M2)
- net M2Z: now also JP11.1; no longer JP11.2
- net OUT1 renamed A1
- net OUT2 renamed A2
- net OUT3 renamed A3
- net R3_RV1: no longer names the net of R3.1, RV1.1
- net RV1_R2: no longer names the net of R2.2, RV1.3
- net SPINDEL_ON_OFF_R_LED: no longer names the net of R4.2, U4.2
- net Spindle_PWM(D5) renamed Analog_0-5V|PWM
- net Analog_0-5V|PWM: now also U7.3 (XTAL2/PB4)
- net Spindle_Speed_Analog_0-5V: no longer names the net of C1.1, JP17.2, R1.2, U1.5 (+)
- net Spindle_Speed_Analog_0-5V: no longer U7.3 (XTAL2/PB4)
- net VDC renamed +VDC
- net VMot renamed VDD
- no-connect marks 13 -> 15
Other:
- note added: "Variable Frequency Drive 0-10V Speed Adjust (VI/ACM Input)\nFrequenzumrichter 0-10V Drehzahleinstellung (VI/ACM Eingang)\n\n"
- note removed: "Variable Frequency Drive 0-10V Speed Control(VI/ACM Input)\nFrequenzumrichter 0-10V Drehzahleinstellung (VI/ACM Eingang)\n\n"
- moved on the sheet: A1, A2, A3, A4, A5, C1, C2, C3, C4, C5, C6, C7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
