File: MPCNC Nano Estlcam Shield.sch (KiCad schematic (older format))
At the start: 92 parts, among them J1 Screw_Terminal_01x02, J10 Conn_01x04_Male, J11 Conn_01x04_Male, J12 Screw_Terminal_01x03, J13 Screw_Terminal_01x03, J14 Screw_Terminal_01x03, J15 Conn_02x03_Odd_Even, J16 Screw_Terminal_01x02, J17 Screw_Terminal_01x02, J18 Screw_Terminal_01x03, J19 Screw_Terminal_01x03, J2 Conn_01x03_Male, J20 Screw_Terminal_01x03, J21 Screw_Terminal_01x03, J22 Screw_Terminal_01x03, J23 Screw_Terminal_01x03, J24 Screw_Terminal_01x03, J25 Screw_Terminal_01x03, J26 Screw_Terminal_01x03, J27 Screw_Terminal_01x03, J28 Conn_01x03_Male, J29 Conn_01x02_Male, J3 Conn_01x06_Male, J4 Screw_Terminal_01x03, J5 Screw_Terminal_01x03, J6 Screw_Terminal_01x03, J7 Conn_01x04_Male, J8 Conn_01x04_Male, J9 Conn_01x04_Male, U1 LM358, U2 LTV-847, U3 LTV-847, U4 LTV-847, U5 ULN2003, U6 L7805, U7 ATtiny45-20PU

Commit message: V1.3
- Version 1.3 of MPCNC Nano Estlcam Shield
   PCB schematic changes:
    # Changed electrolytic capacitor values for L7805 (0,33µF + 0,1µF)
   PCB layout changes:
    # Changed footprint of electrolytic capacitor for L7805 (D=8mm/RM=3,5mm -> D=5mm/RM=2,0mm)
    # Revised heatsink footprint
    + Footprints for many components added to project footprint library ("MPCNC_Shield_Footprints"). Modified footprints from standard KiCad library with value on
silkscreen
    + Added "Uncle Phil" logo on backside silk screen layer
    + Added jumper function description on frontside silk screen layer
    # Changed mounting holes (Edge.cut layer -> footprint)
Parts:
- added H1, H2, H3, H4: MountingHole, MountingHole:MountingHole_4.3mm_M4_DIN965_Pad, symbol Mechanical:MountingHole
- A1: value Arduino_Nano_v3.x -> Arduino Nano
- C1, C2, C3, C4: footprint Capacitor_THT:CP_Radial_D8.0mm_P3.50mm -> MPCNC_Shield_Footprints:CP_Radial_D8.0mm_P3.50mm
- C5: value 1µF -> 0,33µF; footprint Capacitor_THT:CP_Radial_D8.0mm_P3.50mm -> Capacitor_THT:CP_Radial_D5.0mm_P2.00mm
- C6: value 1µF -> 0,1µF; footprint Capacitor_THT:CP_Radial_D8.0mm_P3.50mm -> Capacitor_THT:CP_Radial_D5.0mm_P2.00mm
- D2, D3: footprint Diode_THT:D_DO-201AD_P15.24mm_Horizontal -> MPCNC_Shield_Footprints:D_DO-201AD_P15.24mm_Horizontal
- R1, R10, R11, R12, R13, R14, R15, R16, R17, R18, R2, R3, R4, R5, R6, R7, R8, R9: footprint Resistor_THT:R_Axial_DIN0207_L6.3mm_D2.5mm_P7.62mm_Horizontal -> MPCNC_Shield_Footprints:R_Axial_DIN0207_L6.3mm_D2.5mm_P7.62mm_Horizontal
- U1: footprint Package_DIP:DIP-8_W7.62mm -> MPCNC_Shield_Footprints:DIP-8_W7.62mm
- U2, U3, U4, U5: footprint Package_DIP:DIP-16_W7.62mm -> MPCNC_Shield_Footprints:DIP-16_W7.62mm
- U7: footprint Package_DIP:DIP-8_W7.62mm_LongPads -> MPCNC_Shield_Footprints:DIP-8_W7.62mm
