File: MPCNC Nano Estlcam Shield.sch (KiCad schematic (older format))
At the start: 96 parts, among them J1 Screw_Terminal_01x02, J10 Conn_01x04_Male, J11 Conn_01x04_Male, J12 Screw_Terminal_01x03, J13 Screw_Terminal_01x03, J14 Screw_Terminal_01x03, J15 Conn_02x03_Odd_Even, J16 Screw_Terminal_01x02, J17 Screw_Terminal_01x02, J18 Screw_Terminal_01x03, J19 Screw_Terminal_01x03, J2 Conn_01x03_Male, J20 Screw_Terminal_01x03, J21 Screw_Terminal_01x03, J22 Screw_Terminal_01x03, J23 Screw_Terminal_01x03, J24 Screw_Terminal_01x03, J25 Screw_Terminal_01x03, J26 Screw_Terminal_01x03, J27 Screw_Terminal_01x03, J28 Conn_01x03_Male, J29 Conn_01x02_Male, J3 Conn_01x06_Male, J4 Screw_Terminal_01x03, J5 Screw_Terminal_01x03, J6 Screw_Terminal_01x03, J7 Conn_01x04_Male, J8 Conn_01x04_Male, J9 Conn_01x04_Male, U1 LM358, U2 LTV-847, U3 LTV-847, U4 LTV-847, U5 ULN2003, U6 L7805, U7 ATtiny45-20PU

Commit message: Minor changes for V1.3
   PCB schematic changes:
#Changed footprints for some parts from standard lib to MPCNC lib
   PCB layout changes:
#Added value to silk screen layer for some footprints
Parts:
- C5, C6: footprint Capacitor_THT:CP_Radial_D5.0mm_P2.00mm -> MPCNC_Shield_Footprints:CP_Radial_D5.0mm_P2.00mm
- C7: footprint Capacitor_THT:C_Disc_D3.0mm_W1.6mm_P2.50mm -> MPCNC_Shield_Footprints:C_Disc_D3.0mm_W1.6mm_P2.50mm
- U6: footprint Package_TO_SOT_THT:TO-220-3_Vertical -> MPCNC_Shield_Footprints:TO-220-3_Vertical
Changed lines of the file:
@@
 F 0 "U6" H 12050 3895 50  0000 C CNN
 F 1 "L7805" H 12050 3802 50  0000 C CNN
-F 2 "Package_TO_SOT_THT:TO-220-3_Vertical" H 12075 3500 50  0001 L CIN
+F 2 "MPCNC_Shield_Footprints:TO-220-3_Vertical" H 12075 3500 50  0001 L CIN
 F 3 "http://www.st.com/content/ccc/resource/technical/document/datasheet/41/4f/b3/b0/12/d4/47/88/CD00000444.pdf/files/CD00000444.pdf/jcr:content/translations/en.CD00000444.pdf" H 12050 3600 50  0001 C CNN
 	1    12050 3650
@@
 F 0 "C5" H 11639 3797 50  0000 L CNN
 F 1 "0,33µF" H 11639 3704 50  0000 L CNN
-F 2 "Capacitor_THT:CP_Radial_D5.0mm_P2.00mm" H 11550 3750 50  0001 C CNN
+F 2 "MPCNC_Shield_Footprints:CP_Radial_D5.0mm_P2.00mm" H 11550 3750 50  0001 C CNN
 F 3 "~" H 11550 3750 50  0001 C CNN
 	1    11550 3750
@@
 F 0 "C6" H 12489 3797 50  0000 L CNN
 F 1 "0,1µF" H 12489 3704 50  0000 L CNN
-F 2 "Capacitor_THT:CP_Radial_D5.0mm_P2.00mm" H 12400 3750 50  0001 C CNN
+F 2 "MPCNC_Shield_Footprints:CP_Radial_D5.0mm_P2.00mm" H 12400 3750 50  0001 C CNN
 F 3 "~" H 12400 3750 50  0001 C CNN
 	1    12400 3750
@@
 F 0 "C7" H 11242 7997 50  0000 L CNN
 F 1 "100n" H 11242 7904 50  0000 L CNN
-F 2 "Capacitor_THT:C_Disc_D3.0mm_W1.6mm_P2.50mm" H 11150 7950 50  0001 C CNN
+F 2 "MPCNC_Shield_Footprints:C_Disc_D3.0mm_W1.6mm_P2.50mm" H 11150 7950 50  0001 C CNN
 F 3 "~" H 11150 7950 50  0001 C CNN
 	1    11150 7950

Commit message: V1.4
- Version 1.4 of MPCNC Nano Estlcam Shield
   PCB schematic changes:
    # Changed LED colours (D1:red, D4:green, D5-7:Clear/red)
   PCB layout changes:
    + Footprints for LEDs added to project footprint library ("MPCNC_Shield_Footprints").
    # Changed footprint of LEDs
    # Moved silk screen reference fo L7805 (U6). Reference was hidden by heatsink
    + Added LED 3D models to footprint. LEDs show correct color for 3D model (green, red, white[clear])
    # Changed 3D model for potentiometer (KiCAD standard library model now available in latest KiCAD release 5.10)
    # Changed 3D model for screw terminal blocks (J1; J4-6; J12-14; J16-J17; J18-27)
Parts:
- D1: value LED GREEN -> LED RED; footprint LED_THT:LED_D5.0mm -> MPCNC_Shield_Footprints:LED_D5.0mm_Red
- D4: value LED RED -> LED GREEN; footprint LED_THT:LED_D5.0mm -> MPCNC_Shield_Footprints:LED_D5.0mm_Green
- D5, D6, D7: value LED RED -> LED CLEAR/RED; footprint LED_THT:LED_D3.0mm -> MPCNC_Shield_Footprints:LED_D3.0mm_Clear
Changed lines of the file:
@@
 EESchema Schematic File Version 4
 LIBS:MPCNC Nano Estlcam Shield-cache
-EELAYER 26 0
+EELAYER 29 0
 EELAYER END
 $Descr A3 16535 11693
@@
 Sheet 1 1
 Title "MPCNC Nano Estlcam Shield Schematic"
-Date "2019-03-11"
-Rev "1.3"
+Date "2019-04-16"
+Rev "1.4"
 Comp "T.Nenz"
 Comment1 "Created by:"
@@
 P 12850 4800
 F 0 "D1" V 12935 4681 50  0000 R CNN
-F 1 "LED GREEN" V 12842 4681 50  0000 R CNN
-F 2 "LED_THT:LED_D5.0mm" H 12850 4800 50  0001 C CNN
+F 1 "LED RED" V 12842 4681 50  0000 R CNN
+F 2 "MPCNC_Shield_Footprints:LED_D5.0mm_Red" H 12850 4800 50  0001 C CNN
 F 3 "~" H 12850 4800 50  0001 C CNN
 F 4 "5V Power Indicator " V 12749 4681 50  0000 R CNN "Funktion"
@@
 P 10600 1700
 F 0 "D4" V 10685 1581 50  0000 R CNN
-F 1 "LED RED" V 10592 1581 50  0000 R CNN
-F 2 "LED_THT:LED_D5.0mm" H 10600 1700 50  0001 C CNN
+F 1 "LED GREEN" V 10592 1581 50  0000 R CNN
+F 2 "MPCNC_Shield_Footprints:LED_D5.0mm_Green" H 10600 1700 50  0001 C CNN
 F 3 "~" H 10600 1700 50  0001 C CNN
 F 4 "DC Power Indicator " V 10499 1581 50  0000 R CNN "Funktion"
@@
 P 5400 3700
 F 0 "D6" H 5450 3750 50  0000 R CNN
-F 1 "LED RED" H 5550 3700 50  0000 R CNN
-F 2 "LED_THT:LED_D3.0mm" H 5400 3700 50  0001 C CNN
+F 1 "LED CLEAR/RED" H 5550 3700 50  0000 R CNN
+F 2 "MPCNC_Shield_Footprints:LED_D3.0mm_Clear" H 5400 3700 50  0001 C CNN
 F 3 "~" H 5400 3700 50  0001 C CNN
 F 4 "A2 High" H 5200 3700 50  0000 R CNN "Funktion"
@@
 P 5400 3850
 F 0 "D5" H 5450 3900 50  0000 R CNN
-F 1 "LED RED" H 5550 3850 50  0000 R CNN
-F 2 "LED_THT:LED_D3.0mm" H 5400 3850 50  0001 C CNN
+F 1 "LED CLEAR/RED" H 5550 3850 50  0000 R CNN
+F 2 "MPCNC_Shield_Footprints:LED_D3.0mm_Clear" H 5400 3850 50  0001 C CNN
 F 3 "~" H 5400 3850 50  0001 C CNN
 F 4 "A1 High" H 5200 3850 50  0000 R CNN "Funktion"
@@
 P 5400 3550
 F 0 "D7" H 5400 3600 50  0000 C CNN
-F 1 "LED RED" H 5400 3550 50  0000 C CNN
-F 2 "LED_THT:LED_D3.0mm" H 5400 3550 50  0001 C CNN
+F 1 "LED CLEAR/RED" H 5400 3550 50  0000 C CNN
+F 2 "MPCNC_Shield_Footprints:LED_D3.0mm_Clear" H 5400 3550 50  0001 C CNN
 F 3 "~" H 5400 3550 50  0001 C CNN
 F 4 "A3 High" H 5050 3550 50  0000 C CNN "Funktion"
